File: PCA9685.kicad_sch (KiCad schematic)
At the start: 42 parts, among them U801 PCA9685BS, U802 PCA9685BS

Commit message: daughterboard created
divided into mainboard and daughterboard
Parts:
- removed C801, C802: 10uF, Capacitor_SMD:C_0402_1005Metric, symbol Device:C
- removed R801, R802, R803, R837, R839, R840: 10K, Resistor_SMD:R_0402_1005Metric, symbol Device:R
- removed R804, R806, R823, R824, R825, R826, R827, R828, R829, R830, R831, R832, R833, R834, R835, R836, R841, R842, R843, R844, R845, R846, R847, R848, R849, R850, R851, R852, R853, R854, R855, R856: 220, Resistor_SMD:R_0402_1005Metric, symbol Device:R
- removed U801, U802: PCA9685BS, Package_DFN_QFN:QFN-28-1EP_6x6mm_P0.65mm_EP4.25x4.25mm, symbol Driver_LED:PCA9685BS
